Commit message: Got UDP comms working with SIL in Gazebo

File: rosflight_sim/xacro/fixedwing.urdf.xacro (robot description, xacro)
@@ -62,8 +62,6 @@
   </link>
   <!-- ROSflight_sill -->
-  <xacro:include filename="$(find rosflight_sim)/xacro/ROSflight_SIL.xacro"/>
-  <xacro:generic_fixedwing
-    namespace="${namespace}"
-    parent_link="${namespace}/base_link"/>
+  <xacro:include filename="$(find rosflight_sim)/xacro/rosflight_sil.xacro"/>
+  <xacro:generic_fixedwing namespace="${namespace}" parent_link="${namespace}/base_link"/>
   <!-- Chase Camera
   <xacro:include filename="$(find fcu_sim_plugins)/xacro/camera.xacro"/>

File: rosflight_sim/xacro/multirotor.urdf.xacro (robot description, xacro)
@@ -15,4 +15,5 @@
     <inertia ixx="0.07" ixy="0.0" ixz="0.0" iyy="0.08" iyz="0.0" izz="0.12" />
   </xacro:property>
+  <xacro:property name="color" value="White" />
   <!-- *********************** GAZEBO ROBOT DEFINITION ******************* -->
   <link name="${namespace}/base_link">
@@ -41,8 +42,8 @@
   </link>
   <gazebo reference="${namespace}/base_link">
-    <material>Gazebo/$(arg color)</material>
+    <material>Gazebo/${color}</material>
   </gazebo>
-  <!-- ROSflight_SIL -->
-  <xacro:include filename="$(find rosflight_sim)/xacro/ROSflight_SIL.xacro"/>
+  <!-- ROSflight SIL Plugin -->
+  <xacro:include filename="$(find rosflight_sim)/xacro/rosflight_sil.xacro"/>
   <xacro:generic_multirotor namespace="${namespace}" parent_link="${namespace}/base_link"/>
 </robot>

Commit message: fixed #24

File: rosflight_sim/xacro/fixedwing.urdf.xacro (robot description, xacro)
@@ -7,9 +7,8 @@
   <!-- Properties -->
   <xacro:property name="namespace" value="fixedwing"/>
-  <xacro:property name="wind_speed_topic" value="gazebo/wind_speed"/>
   <xacro:property name="use_mesh_file" value="true" />
   <xacro:property name="mesh_file" value="model://zephyr_delta_wing/meshes/wing.dae"/>
   <xacro:property name="body_width" value="1.4"/>
-  <xacro:property name="body_height" value="1.0" />
+  <xacro:property name="body_height" value="0.3" />
   <xacro:property name="body_length" value="1.6"/>
   <xacro:property name="mass" value="1.5"/>
@@ -18,8 +17,4 @@
   <xacro:property name="Jz" value="0.1712"/>
   <xacro:property name="Jxz" value="0.0015"/>
-  <!-- Property Blocks -->
-  <xacro:property name="empty_inertia">
-    <inertia ixx="0.0001" ixy="0.0" ixz="0.0" iyy="0.0001" iyz="0.0" izz="0.001" />
-  </xacro:property>
   <!-- Instantiate Link and Visual -->
   <link name="${namespace}/base_link">
@@ -41,25 +36,11 @@
     </visual>
     <collision name="plane_collision">
-      <origin xyz="0 0 0" rpy="1.570796 0 1.570796" />
+      <origin xyz="0 0 0" rpy="0 0 0" />
       <geometry>
-        <box size="${body_width} ${body_height} ${body_length}" />
+        <cylinder length="${body_height}" radius="${body_width}"/>
       </geometry>
     </collision>
-    <!-- Wheels
-    <xacro:include filename="$(find fcu_sim_plugins)/xacro/wheel.xacro"/>
-    <xacro:caster
-      radius="0.05">
-      <origin xyz="${body_length*0.5} -${body_width*0.5} -${body_height*0.5}"/>
-    </xacro:caster>
-    <xacro:caster
-      radius="0.05">
-      <origin xyz="${body_length*0.5} ${body_width*0.5} -${body_height*0.5}"/>
-    </xacro:caster>
-    <xacro:caster
-      radius="0.05">
-      <origin xyz="-${body_length*0.5} 0 -${body_height*0.4}"/>
-    </xacro:caster> -->
   </link>
-  <!-- ROSflight_sill -->
+  <!-- ROSflight SIL Plugin -->
   <xacro:include filename="$(find rosflight_sim)/xacro/rosflight_sil.xacro"/>
   <xacro:generic_fixedwing namespace="${namespace}" parent_link="${namespace}/base_link"/>

Commit message: a little cleanup

File: rosflight_sim/xacro/fixedwing.urdf.xacro (robot description, xacro)
@@ -45,18 +45,3 @@
   <xacro:include filename="$(find rosflight_sim)/xacro/rosflight_sil.xacro"/>
   <xacro:generic_fixedwing namespace="${namespace}" parent_link="${namespace}/base_link"/>
-  <!-- Chase Camera
-  <xacro:include filename="$(find fcu_sim_plugins)/xacro/camera.xacro"/>
-  <xacro:simple_camera
-    namespace="${namespace}/chase"
-    frame_rate="30"
-    rgb_range="1000"
-    parent_link="${namespace}/base_link"
-    image_topic="rgb"
-    image_camera_info_topic="camera_info">
-    <origin xyz="-${1.1*body_length} 0 ${0.8*body_height}"/>
-  </xacro:simple_camera> -->
-  <!-- Color
-  <gazebo reference="${namespace}/base_link">
-    <material>Gazebo/Blue</material>
-  </gazebo> -->
 </robot>

Commit message: Got fixedwing launching and cleaned up parameters

File: rosflight_sim/xacro/fixedwing.urdf.xacro (robot description, xacro)
@@ -8,5 +8,5 @@
   <xacro:property name="namespace" value="fixedwing"/>
   <xacro:property name="use_mesh_file" value="true" />
-  <xacro:property name="mesh_file" value="model://zephyr_delta_wing/meshes/wing.dae"/>
+  <xacro:property name="mesh_file" value="$(arg mesh_file_location)" />
   <xacro:property name="body_width" value="1.4"/>
   <xacro:property name="body_height" value="0.3" />

Commit message: Removed unused mass and inertia definitions

File: rosflight_sim/xacro/fixedwing.urdf.xacro (robot description, xacro)
@@ -12,9 +12,9 @@
   <xacro:property name="body_height" value="0.3" />
   <xacro:property name="body_length" value="1.6"/>
-  <xacro:property name="mass" value="1.5"/>
-  <xacro:property name="Jx" value="0.1147"/>
-  <xacro:property name="Jy" value="0.0576"/>
-  <xacro:property name="Jz" value="0.1712"/>
-  <xacro:property name="Jxz" value="0.0015"/>
+  <xacro:property name="mass" value="3.92"/>
+  <xacro:property name="Jx" value="0.213"/>
+  <xacro:property name="Jy" value="0.171"/>
+  <xacro:property name="Jz" value="0.350"/>
+  <xacro:property name="Jxz" value="0.04"/>
   <!-- Instantiate Link and Visual -->
   <link name="${namespace}/base_link">

File: rosflight_sim/xacro/multirotor.urdf.xacro (robot description, xacro)
@@ -10,5 +10,5 @@
   <xacro:property name="use_mesh_file" value="true" />
   <xacro:property name="mesh_file" value="$(arg mesh_file_location)" />
-  <xacro:property name="mass" value="2.856" />
+  <xacro:property name="mass" value="2.0" />
   <xacro:property name="body_width" value="0.505" />
   <xacro:property name="body_height" value="0.1" />

Commit message: Update code to match ROS2 style guide

File: rosflight_sim/xacro/fixedwing.urdf.xacro (robot description, xacro)
@@ -4,11 +4,11 @@
 Author: Gary Ellingson
 -->
-<robot name="fixedwing" xmlns:xacro="http://ros.org/wiki/xacro">
+<robot xmlns:xacro="http://ros.org/wiki/xacro" name="fixedwing">
   <!-- Properties -->
   <xacro:property name="namespace" value="fixedwing"/>
-  <xacro:property name="use_mesh_file" value="true" />
-  <xacro:property name="mesh_file" value="$(arg mesh_file_location)" />
+  <xacro:property name="use_mesh_file" value="true"/>
+  <xacro:property name="mesh_file" value="$(arg mesh_file_location)"/>
   <xacro:property name="body_width" value="1.4"/>
-  <xacro:property name="body_height" value="0.3" />
+  <xacro:property name="body_height" value="0.3"/>
   <xacro:property name="body_length" value="1.6"/>
   <xacro:property name="mass" value="3.92"/>
@@ -20,21 +20,21 @@
   <link name="${namespace}/base_link">
     <inertial>
-      <mass value="${mass}" />
-      <origin xyz="0 0 0" />
-      <inertia ixx="${Jx}" ixy="0.00" ixz="${Jxz}" iyy="${Jy}" iyz="0.00" izz="${Jz}" />
+      <mass value="${mass}"/>
+      <origin xyz="0 0 0"/>
+      <inertia ixx="${Jx}" ixy="0.00" ixz="${Jxz}" iyy="${Jy}" iyz="0.00" izz="${Jz}"/>
     </inertial>
     <visual name="plane_visual">
-      <origin xyz="0 0 0" rpy="0 0 1.570796" />
+      <origin xyz="0 0 0" rpy="0 0 1.570796"/>
       <geometry>
         <xacro:if value="${use_mesh_file}">
-          <mesh filename="${mesh_file}" scale="1 1 1" />
+          <mesh filename="${mesh_file}" scale="1 1 1"/>
         </xacro:if>
         <xacro:unless value="${use_mesh_file}">
-            <box size="${body_width} ${body_height} ${body_length}" />
+          <box size="${body_width} ${body_height} ${body_length}"/>
         </xacro:unless>
       </geometry>
     </visual>
     <collision name="plane_collision">
-      <origin xyz="0 0 0" rpy="0 0 0" />
+      <origin xyz="0 0 0" rpy="0 0 0"/>
       <geometry>
         <cylinder length="${body_height}" radius="${body_width}"/>

File: rosflight_sim/xacro/multirotor.urdf.xacro (robot description, xacro)
@@ -4,28 +4,29 @@
 Author: James Jackson
 -->
-<robot name="multirotor" xmlns:xacro="http://ros.org/wiki/xacro">
+<robot xmlns:xacro="http://ros.org/wiki/xacro" name="multirotor">
   <!-- Properties -->
   <xacro:arg name="mav_name" default="multirotor"/>
-  <xacro:property name="namespace" value="$(arg mav_name)" />
-  <xacro:property name="use_mesh_file" value="true" />
-  <xacro:property name="mesh_file" value="$(arg mesh_file_location)" />
-  <xacro:property name="mass" value="2.0" />
-  <xacro:property name="body_width" value="0.505" />
-  <xacro:property name="body_height" value="0.1" />
+  <xacro:property name="namespace" value="$(arg mav_name)"/>
+  <xacro:property name="use_mesh_file" value="true"/>
+  <xacro:property name="mesh_file" value="$(arg mesh_file_location)"/>
+  <xacro:property name="mass" value="2.0"/>
+  <xacro:property name="body_width" value="0.505"/>
+  <xacro:property name="body_height" value="0.1"/>
   <xacro:property name="body_inertia">
-    <inertia ixx="0.07" ixy="0.0" ixz="0.0" iyy="0.08" iyz="0.0" izz="0.12" />
-  </xacro:property> />
+    <inertia ixx="0.07" ixy="0.0" ixz="0.0" iyy="0.08" iyz="0.0" izz="0.12"/>
+  </xacro:property>
+  />
   <!-- *********************** GAZEBO ROBOT DEFINITION ******************* -->
   <link name="${namespace}/base_link">
     <inertial>
-      <mass value="${mass}" />  <!-- [kg] -->
-      <origin xyz="0 0 0" />
-      <xacro:insert_block name="body_inertia" />
+      <mass value="${mass}"/>  <!-- [kg] -->
+      <origin xyz="0 0 0"/>
+      <xacro:insert_block name="body_inertia"/>
     </inertial>
     <visual>
-      <origin xyz="0 0 0" rpy="0 0 0" />
+      <origin xyz="0 0 0" rpy="0 0 0"/>
       <geometry>
         <xacro:if value="${use_mesh_file}">
-          <mesh filename="${mesh_file}" scale="1 1 1" />
+          <mesh filename="${mesh_file}" scale="1 1 1"/>
         </xacro:if>
         <xacro:unless value="${use_mesh_file}">
@@ -35,8 +36,8 @@
     </visual>
     <collision>
-      <origin xyz="0 0 0" rpy="0 0 0" />
+      <origin xyz="0 0 0" rpy="0 0 0"/>
       <geometry>
         <xacro:if value="${use_mesh_file}">
-          <mesh filename="${mesh_file}" scale="1 1 1" />
+          <mesh filename="${mesh_file}" scale="1 1 1"/>
         </xacro:if>
         <xacro:unless value="${use_mesh_file}">

File: rosflight_sim/xacro/rosflight_sil.xacro (robot description, xacro)
@@ -18,5 +18,5 @@
   <!-- Macro to add a rosflight_sil plugin. -->
   <xacro:macro name="rosflight_sil_plugin"
-    params="namespace parent_link mav_type parent_frame_id">
+               params="namespace parent_link mav_type parent_frame_id">
     <gazebo>
       <plugin filename="librosflight_sil_plugin.so" name="rosflight_sil">

Commit message: Polished up sim params

File: rosflight_sim/xacro/fixedwing.urdf.xacro (robot description, xacro)
@@ -12,8 +12,8 @@
   <xacro:property name="body_height" value="0.3"/>
   <xacro:property name="body_length" value="1.6"/>
-  <xacro:property name="mass" value="3.92"/>
-  <xacro:property name="Jx" value="0.213"/>
-  <xacro:property name="Jy" value="0.171"/>
-  <xacro:property name="Jz" value="0.350"/>
+  <xacro:property name="mass" value="2.28"/>
+  <xacro:property name="Jx" value="0.141"/>
+  <xacro:property name="Jy" value="0.208"/>
+  <xacro:property name="Jz" value="0.293"/>
   <xacro:property name="Jxz" value="0.04"/>
   <!-- Instantiate Link and Visual -->

Commit message: Fixed 3D model scaling issues and added texture.

File: rosflight_sim/xacro/fixedwing.urdf.xacro (robot description, xacro)
@@ -9,7 +9,7 @@
   <xacro:property name="use_mesh_file" value="true"/>
   <xacro:property name="mesh_file" value="$(arg mesh_file_location)"/>
-  <xacro:property name="body_width" value="1.4"/>
-  <xacro:property name="body_height" value="0.3"/>
-  <xacro:property name="body_length" value="1.6"/>
+  <xacro:property name="body_width" value="1.8"/>
+  <xacro:property name="body_height" value="0.1778"/>
+  <xacro:property name="body_length" value="1.27"/>
   <xacro:property name="mass" value="2.28"/>
   <xacro:property name="Jx" value="0.141"/>
