Commit message: removed skyhunter, added aerosonde

File: rosflight_sim/xacro/aerosonde.urdf.xacro (robot description, xacro)
@@ -12,9 +12,9 @@
   <xacro:property name="body_height" value="0.1778"/>
   <xacro:property name="body_length" value="1.27"/>
-  <xacro:property name="mass" value="2.28"/>
-  <xacro:property name="Jx" value="0.141"/>
-  <xacro:property name="Jy" value="0.208"/>
-  <xacro:property name="Jz" value="0.293"/>
-  <xacro:property name="Jxz" value="0.04"/>
+  <xacro:property name="mass" value="11.0"/>
+  <xacro:property name="Jx" value="0.8224"/>
+  <xacro:property name="Jy" value="1.135"/>
+  <xacro:property name="Jz" value="1.759"/>
+  <xacro:property name="Jxz" value="0.1204"/>
   <!-- Instantiate Link and Visual -->
   <link name="${namespace}/base_link">
