Commit message: some tweaks to make multi-agent possible

File: rosflight_sim/xacro/multirotor.urdf.xacro (robot description, xacro)
@@ -6,5 +6,7 @@
 <robot name="multirotor" xmlns:xacro="http://ros.org/wiki/xacro">
   <!-- Properties -->
-  <xacro:property name="namespace" value="multirotor" />
+  <xacro:arg name="mav_name" default="multirotor"/>
+  <xacro:arg name="color" default="White"/>
+  <xacro:property name="namespace" value="$(arg mav_name)" />
   <xacro:property name="use_mesh_file" value="true" />
   <xacro:property name="mesh_file" value="model://quadrotor/meshes/quadrotor_base.dae" />
@@ -15,5 +17,5 @@
     <inertia ixx="0.07" ixy="0.0" ixz="0.0" iyy="0.08" iyz="0.0" izz="0.12" />
   </xacro:property>
-  <xacro:property name="color" value="White" />
+  <xacro:property name="color" value="$(arg color)" />
   <!-- *********************** GAZEBO ROBOT DEFINITION ******************* -->
   <link name="${namespace}/base_link">

Commit message: Got gazebo model loading

File: rosflight_sim/xacro/multirotor.urdf.xacro (robot description, xacro)
@@ -10,5 +10,5 @@
   <xacro:property name="namespace" value="$(arg mav_name)" />
   <xacro:property name="use_mesh_file" value="true" />
-  <xacro:property name="mesh_file" value="model://quadrotor/meshes/quadrotor_base.dae" />
+  <xacro:property name="mesh_file" value="$(arg mesh_file_location)" />
   <xacro:property name="mass" value="2.856" />
   <xacro:property name="body_width" value="0.505" />

Commit message: Cleaned up multirotor launch file

File: rosflight_sim/xacro/multirotor.urdf.xacro (robot description, xacro)
@@ -7,5 +7,4 @@
   <!-- Properties -->
   <xacro:arg name="mav_name" default="multirotor"/>
-  <xacro:arg name="color" default="White"/>
   <xacro:property name="namespace" value="$(arg mav_name)" />
   <xacro:property name="use_mesh_file" value="true" />
@@ -16,6 +15,5 @@
   <xacro:property name="body_inertia">
     <inertia ixx="0.07" ixy="0.0" ixz="0.0" iyy="0.08" iyz="0.0" izz="0.12" />
-  </xacro:property>
-  <xacro:property name="color" value="$(arg color)" />
+  </xacro:property> />
   <!-- *********************** GAZEBO ROBOT DEFINITION ******************* -->
   <link name="${namespace}/base_link">
@@ -44,5 +42,4 @@
   </link>
   <gazebo reference="${namespace}/base_link">
-    <material>Gazebo/${color}</material>
   </gazebo>
   <!-- ROSflight SIL Plugin -->

Commit message: Added multirotor world (asphalt) and improved collision

File: rosflight_sim/xacro/multirotor.urdf.xacro (robot description, xacro)
@@ -37,5 +37,10 @@
       <origin xyz="0 0 0" rpy="0 0 0" />
       <geometry>
-        <cylinder length="${body_height}" radius="${body_width}"/>
+        <xacro:if value="${use_mesh_file}">
+          <mesh filename="${mesh_file}" scale="1 1 1" />
+        </xacro:if>
+        <xacro:unless value="${use_mesh_file}">
+          <cylinder length="${body_height}" radius="${body_width}"/>
+        </xacro:unless>
       </geometry>
     </collision>

Commit message: Fixed thrust coeffs, updated drag model and mass.
Working model that reflects reality relativley well. The params are
hardcoded in this commit.

File: rosflight_sim/xacro/multirotor.urdf.xacro (robot description, xacro)
@@ -10,9 +10,9 @@
   <xacro:property name="use_mesh_file" value="true"/>
   <xacro:property name="mesh_file" value="$(arg mesh_file_location)"/>
-  <xacro:property name="mass" value="2.0"/>
+  <xacro:property name="mass" value="3.5"/>
   <xacro:property name="body_width" value="0.505"/>
   <xacro:property name="body_height" value="0.1"/>
   <xacro:property name="body_inertia">
-    <inertia ixx="0.07" ixy="0.0" ixz="0.0" iyy="0.08" iyz="0.0" izz="0.12"/>
+    <inertia ixx="0.08" ixy="0.0" ixz="0.0" iyy="0.08" iyz="0.0" izz="0.12"/>
   </xacro:property>
   />
