Commit message: feat: Small fixes to comments based on code review discussion, renaming variables and files, and converting transformations to Eigen transformations

File: rosflight_sim/simulators/gazebo_sim/xacro/rosflight_sil.xacro (robot description, xacro)
@@ -3,5 +3,5 @@
   <!-- Forces And Moments Plugin -->
   <xacro:macro name="generic_multirotor" params="namespace parent_link">
-    <xacro:rosflight_sil_plugin
+    <xacro:gazebo_dynamics_plugin
       namespace="${namespace}"
       parent_link="${namespace}/base_link"
@@ -10,5 +10,5 @@
   </xacro:macro>
   <xacro:macro name="generic_fixedwing" params="namespace parent_link">
-    <xacro:rosflight_sil_plugin
+    <xacro:gazebo_dynamics_plugin
       namespace="${namespace}"
       parent_link="${namespace}/base_link"
@@ -17,5 +17,5 @@
   </xacro:macro>
   <!-- Macro to add a gazebo_dynamics plugin. -->
-  <xacro:macro name="rosflight_sil_plugin"
+  <xacro:macro name="gazebo_dynamics_plugin"
                params="namespace parent_link mav_type parent_frame_id">
     <gazebo>
